File: kicad/a2k6-cart.kicad_pcb (KiCad board)
At the start: 2 copper layers, 41.4 x 51.7 mm, 2 parts, among them J1 2600_Cartridge_Port, J2 Conn_02x12

Commit message: Updating project name
Other:
- board text added: "Selecta Adapter"
- board text added: "github.com/kevinl95/atari2600-selecta2600-adapter"
- board text removed: "A2k6 Cartridge"
- board text removed: "github.com/sarweiler/a2k6-cart"
Changed lines of the file:
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@@
 		(layer "Edge.Cuts")
 	)
-	(gr_text "github.com/sarweiler/a2k6-cart"
-		(at 132.842 93.472 90)
+	(gr_text "github.com/kevinl95/atari2600-selecta2600-adapter"
+		(at 136 92.5 90)
 		(layer "B.SilkS")
 		(effects
@@
 		)
 	)
-	(gr_text "A2k6 Cartridge"
-		(at 133.096 92.964 90)
+	(gr_text "Selecta Adapter"
+		(at 133.5 94 90)
 		(layer "F.SilkS")
 		(effects
