File: kicad/a2k6-cart.kicad_sch (KiCad schematic)
At the start: 2 parts, among them J1 2600_Cartridge_Port, J2 Conn_02x12

Commit message: Updating project name
Other:
- title: Selectra2600 Ribbon Cable Adapter -> Selecta2600 Ribbon Cable Adapter
- moved on the sheet: J1
